Commit message: Updating moveit demo to allow trajectory execution in gazebo

File: ros/kuka_lwr/lwr_description/robot/lwr_on_box.urdf.xacro (robot description, xacro)
@@ -30,5 +30,5 @@
 	</gazebo>
 	<xacro:kuka_lwr parent="world" name="lwr">
-		<origin xyz="0 0 0" rpy="0 0 0"/>
+		<origin xyz="0 0 1" rpy="0 0 0"/>
 	</xacro:kuka_lwr>
 </robot>
