Commit message: edited to make it INDIGO compatible

File: ros/kuka_lwr/lwr_description/model/kuka_lwr.transmission.xacro (robot description, xacro)
@@ -4,5 +4,7 @@
 	    <transmission name="${name}_arm_0_trans">
 			<type>transmission_interface/SimpleTransmission</type>
-			<joint name="${name}_arm_0_joint"/>
+			<joint name="${name}_arm_0_joint">
+				<hardwareInterface>EffortJointInterface</hardwareInterface>
+			</joint>
 			<actuator name="${name}_arm_0_motor">
 				<hardwareInterface>EffortJointInterface</hardwareInterface>
@@ -12,5 +14,7 @@
 		<transmission name="${name}_arm_1_trans">
 			<type>transmission_interface/SimpleTransmission</type>
-			<joint name="${name}_arm_1_joint"/>
+			<joint name="${name}_arm_1_joint">
+				<hardwareInterface>EffortJointInterface</hardwareInterface>
+			</joint>
 			<actuator name="${name}_arm_1_motor">
 				<hardwareInterface>EffortJointInterface</hardwareInterface>
@@ -20,5 +24,7 @@
 		<transmission name="${name}_arm_2_trans">
 			<type>transmission_interface/SimpleTransmission</type>
-			<joint name="${name}_arm_2_joint"/>
+			<joint name="${name}_arm_2_joint">
+				<hardwareInterface>EffortJointInterface</hardwareInterface>
+			</joint>
 			<actuator name="${name}_arm_2_motor">
 				<hardwareInterface>EffortJointInterface</hardwareInterface>
@@ -28,5 +34,7 @@
 		<transmission name="${name}_arm_3_trans">
 			<type>transmission_interface/SimpleTransmission</type>
-			<joint name="${name}_arm_3_joint"/>
+			<joint name="${name}_arm_3_joint">
+				<hardwareInterface>EffortJointInterface</hardwareInterface>
+			</joint>
 			<actuator name="${name}_arm_3_motor">
 				<hardwareInterface>EffortJointInterface</hardwareInterface>
@@ -36,5 +44,7 @@
 		<transmission name="${name}_arm_4_trans">
 			<type>transmission_interface/SimpleTransmission</type>
-			<joint name="${name}_arm_4_joint"/>
+			<joint name="${name}_arm_4_joint">
+				<hardwareInterface>EffortJointInterface</hardwareInterface>
+			</joint>
 			<actuator name="${name}_arm_4_motor">
 				<hardwareInterface>EffortJointInterface</hardwareInterface>
@@ -44,5 +54,7 @@
 		<transmission name="${name}_arm_5_trans">
 			<type>transmission_interface/SimpleTransmission</type>
-			<joint name="${name}_arm_5_joint"/>
+			<joint name="${name}_arm_5_joint">
+				<hardwareInterface>EffortJointInterface</hardwareInterface>
+			</joint>
 			<actuator name="${name}_arm_5_motor">
 				<hardwareInterface>EffortJointInterface</hardwareInterface>
@@ -52,5 +64,7 @@
 		<transmission name="${name}_arm_6_trans">
 			<type>transmission_interface/SimpleTransmission</type>
-			<joint name="${name}_arm_6_joint"/>
+			<joint name="${name}_arm_6_joint">
+				<hardwareInterface>EffortJointInterface</hardwareInterface>
+			</joint>
 			<actuator name="${name}_arm_6_motor">
 				<hardwareInterface>EffortJointInterface</hardwareInterface>
