Commit message: lauch files parameterized to enable multiple robot setup

File: ros/kuka_lwr/lwr_description/model/kuka_lwr.gazebo.xacro (robot description, xacro)
@@ -2,39 +2,39 @@
 <robot xmlns:xacro="http://ros.org/wiki/xacro">
 	<xacro:macro name="kuka_lwr_gazebo" params="name">
-		<gazebo>
-			<plugin name="gazebo_ros_control" filename="libgazebo_ros_control.so">
-				<robotNamespace>/lwr</robotNamespace>
-			</plugin>
-		</gazebo>
-		<gazebo reference="calib_${name}_arm_base_link">
-			<gravity>true</gravity>
+<!-- 		<gazebo>
+			<plugin name="gazebo_ros_control" filename="libgazebo_ros_control.so"> -->
+				<!-- <robotNamespace>/lwr</robotNamespace> -->
+<!-- 			</plugin>
+		</gazebo> -->
+		<gazebo reference="${name}_arm_base_link">
+			<!-- <gravity>true</gravity> -->
 			<material>Gazebo/Orange</material>
 		</gazebo>
 		<gazebo reference="${name}_arm_1_link">
-			<gravity>true</gravity>
+			<!-- <gravity>true</gravity> -->
 			<material>Gazebo/Orange</material>
 		</gazebo>
 		<gazebo reference="${name}_arm_2_link">
-			<gravity>true</gravity>
+			<!-- <gravity>true</gravity> -->
 			<material>Gazebo/Orange</material>
 		</gazebo>
 		<gazebo reference="${name}_arm_3_link">
-			<gravity>true</gravity>
+			<!-- <gravity>true</gravity> -->
 			<material>Gazebo/Orange</material>
 		</gazebo>
 		<gazebo reference="${name}_arm_4_link">
-			<gravity>true</gravity>
+			<!-- <gravity>true</gravity> -->
 			<material>Gazebo/Orange</material>
 		</gazebo>
 		<gazebo reference="${name}_arm_5_link">
-			<gravity>true</gravity>
+			<!-- <gravity>true</gravity> -->
 			<material>Gazebo/Orange</material>
 		</gazebo>
 		<gazebo reference="${name}_arm_6_link">
-			<gravity>true</gravity>
+			<!-- <gravity>true</gravity> -->
 			<material>Gazebo/Orange</material>
 		</gazebo>
 		<gazebo reference="${name}_arm_7_link">
-			<gravity>true</gravity>
+			<!-- <gravity>true</gravity> -->
 			<material>Gazebo/Grey</material>
 		</gazebo>

File: ros/kuka_lwr/lwr_description/model/kuka_lwr.urdf.xacro (robot description, xacro)
@@ -1,4 +1,4 @@
 <?xml version="1.0"?>
-<robot xmlns:xacro="http://www.ros.org/wiki/xacro">
+<robot name="kuka_lwr" xmlns:xacro="http://www.ros.org/wiki/xacro">
 	<!-- utils /-->
 	<xacro:include filename="$(find lwr_description)/model/utils.xacro"/>
@@ -19,7 +19,7 @@
 		<origin xyz="0 0 0" rpy="0 0 0"/>
 		<parent link="${parent}"/>
-		<child link="calib_${name}_arm_base_link"/>
-	</joint>
-	<link name="calib_${name}_arm_base_link">
+		<child link="${name}_arm_base_link"/>
+	</joint>
+	<link name="${name}_arm_base_link">
 		<inertial>
 			<mass value="${base_mass}"/>
@@ -49,5 +49,5 @@
 		<safety_controller soft_lower_limit="${-168 * M_PI / 180}" soft_upper_limit="${168 * M_PI / 180}" k_position="30" k_velocity="30"/>
 		<dynamics damping="1.0"/>
-		<parent link="calib_${name}_arm_base_link"/>
+		<parent link="${name}_arm_base_link"/>
 		<child link="${name}_arm_1_link"/>
 	</joint>

File: ros/kuka_lwr/lwr_description/robot/lwr_on_box.urdf.xacro (robot description, xacro)
@@ -2,4 +2,9 @@
 <robot xmlns:xacro="http://www.ros.org/wiki/xacro" name="lwr">
 	<xacro:include filename="$(find lwr_description)/model/kuka_lwr.urdf.xacro"/>
+	<gazebo>
+		<plugin name="gazebo_ros_control" filename="libgazebo_ros_control.so">
+			<!-- <robotNamespace>/lwr</robotNamespace> -->
+		</plugin>
+	</gazebo>
 	<link name="world">
 		<!-- <inertial>
@@ -25,5 +30,5 @@
 	</gazebo>
 	<xacro:kuka_lwr parent="world" name="lwr">
-		<origin xyz="0 0 1.0" rpy="0 0 0"/>
+		<origin xyz="0 0 0" rpy="0 0 0"/>
 	</xacro:kuka_lwr>
 </robot>

Commit message: Fix in kuka_controllers CMakeLists.txt file. Gazebo/ROS control plugin namespace dependant.

File: ros/kuka_lwr/lwr_description/model/kuka_lwr.gazebo.xacro (robot description, xacro)
@@ -2,9 +2,9 @@
 <robot xmlns:xacro="http://ros.org/wiki/xacro">
 	<xacro:macro name="kuka_lwr_gazebo" params="name">
-<!-- 		<gazebo>
-			<plugin name="gazebo_ros_control" filename="libgazebo_ros_control.so"> -->
-				<!-- <robotNamespace>/lwr</robotNamespace> -->
-<!-- 			</plugin>
-		</gazebo> -->
+		<gazebo>
+			<plugin name="gazebo_ros_control" filename="libgazebo_ros_control.so">
+				<robotNamespace>${name}</robotNamespace>
+			</plugin>
+		</gazebo>
 		<gazebo reference="${name}_arm_base_link">
 			<gravity>true</gravity>

File: ros/kuka_lwr/lwr_description/robot/lwr_on_box.urdf.xacro (robot description, xacro)
@@ -2,15 +2,10 @@
 <robot xmlns:xacro="http://www.ros.org/wiki/xacro" name="lwr">
 	<xacro:include filename="$(find lwr_description)/model/kuka_lwr.urdf.xacro"/>
-	<gazebo>
-		<plugin name="gazebo_ros_control" filename="libgazebo_ros_control.so">
-			<!-- <robotNamespace>/lwr</robotNamespace> -->
-		</plugin>
-	</gazebo>
 	<link name="world">
-		<!-- <inertial>
+		<inertial>
 			<mass value="50.0"/>
 			<com xyz="0 0 0"/>
 			<inertia  ixx="0.01" ixy="0.00"  ixz="0.00" iyy="0.01" iyz="0.00" izz="0.01" />
-		</inertial> -->
+		</inertial>
 		<visual>
 			<origin xyz="0 0 0.50" rpy="0 0 0"/>

Commit message: updating the lwr_hw, update the urdf to delete the word _arm at every joint and link

File: ros/kuka_lwr/lwr_description/model/kuka_lwr.gazebo.xacro (robot description, xacro)
@@ -7,33 +7,33 @@
 			</plugin>
 		</gazebo>
-		<gazebo reference="${name}_arm_base_link">
+		<gazebo reference="${name}_base_link">
 			<gravity>true</gravity>
 			<material>Gazebo/Orange</material>
 		</gazebo>
-		<gazebo reference="${name}_arm_1_link">
+		<gazebo reference="${name}_1_link">
 			<gravity>true</gravity>
 			<material>Gazebo/Orange</material>
 		</gazebo>
-		<gazebo reference="${name}_arm_2_link">
+		<gazebo reference="${name}_2_link">
 			<gravity>true</gravity>
 			<material>Gazebo/Orange</material>
 		</gazebo>
-		<gazebo reference="${name}_arm_3_link">
+		<gazebo reference="${name}_3_link">
 			<gravity>true</gravity>
 			<material>Gazebo/Orange</material>
 		</gazebo>
-		<gazebo reference="${name}_arm_4_link">
+		<gazebo reference="${name}_4_link">
 			<gravity>true</gravity>
 			<material>Gazebo/Orange</material>
 		</gazebo>
-		<gazebo reference="${name}_arm_5_link">
+		<gazebo reference="${name}_5_link">
 			<gravity>true</gravity>
 			<material>Gazebo/Orange</material>
 		</gazebo>
-		<gazebo reference="${name}_arm_6_link">
+		<gazebo reference="${name}_6_link">
 			<gravity>true</gravity>
 			<material>Gazebo/Orange</material>
 		</gazebo>
-		<gazebo reference="${name}_arm_7_link">
+		<gazebo reference="${name}_7_link">
 			<gravity>true</gravity>
 			<material>Gazebo/Grey</material>

File: ros/kuka_lwr/lwr_description/model/kuka_lwr.transmission.xacro (robot description, xacro)
@@ -2,70 +2,70 @@
 <robot xmlns:xacro="http://ros.org/wiki/xacro">
     <xacro:macro name="kuka_lwr_transmission" params="name">
-	    <transmission name="${name}_arm_0_trans">
+	    <transmission name="${name}_0_trans">
 			<type>transmission_interface/SimpleTransmission</type>
-			<joint name="${name}_arm_0_joint">
+			<joint name="${name}_0_joint">
 				<hardwareInterface>EffortJointInterface</hardwareInterface>
 			</joint>
-			<actuator name="${name}_arm_0_motor">
+			<actuator name="${name}_0_motor">
 				<hardwareInterface>EffortJointInterface</hardwareInterface>
 				<mechanicalReduction>1</mechanicalReduction>
 			</actuator>
 	    </transmission>
-		<transmission name="${name}_arm_1_trans">
+		<transmission name="${name}_1_trans">
 			<type>transmission_interface/SimpleTransmission</type>
-			<joint name="${name}_arm_1_joint">
+			<joint name="${name}_1_joint">
 				<hardwareInterface>EffortJointInterface</hardwareInterface>
 			</joint>
-			<actuator name="${name}_arm_1_motor">
+			<actuator name="${name}_1_motor">
 				<hardwareInterface>EffortJointInterface</hardwareInterface>
 				<mechanicalReduction>1</mechanicalReduction>
 			</actuator>
 		</transmission>
-		<transmission name="${name}_arm_2_trans">
+		<transmission name="${name}_2_trans">
 			<type>transmission_interface/SimpleTransmission</type>
-			<joint name="${name}_arm_2_joint">
+			<joint name="${name}_2_joint">
 				<hardwareInterface>EffortJointInterface</hardwareInterface>
 			</joint>
-			<actuator name="${name}_arm_2_motor">
+			<actuator name="${name}_2_motor">
 				<hardwareInterface>EffortJointInterface</hardwareInterface>
 				<mechanicalReduction>1</mechanicalReduction>
 			</actuator>
 		</transmission>
-		<transmission name="${name}_arm_3_trans">
+		<transmission name="${name}_3_trans">
 			<type>transmission_interface/SimpleTransmission</type>
-			<joint name="${name}_arm_3_joint">
+			<joint name="${name}_3_joint">
 				<hardwareInterface>EffortJointInterface</hardwareInterface>
 			</joint>
-			<actuator name="${name}_arm_3_motor">
+			<actuator name="${name}_3_motor">
 				<hardwareInterface>EffortJointInterface</hardwareInterface>
 				<mechanicalReduction>1</mechanicalReduction>
 			</actuator>
 		</transmission>
-		<transmission name="${name}_arm_4_trans">
+		<transmission name="${name}_4_trans">
 			<type>transmission_interface/SimpleTransmission</type>
-			<joint name="${name}_arm_4_joint">
+			<joint name="${name}_4_joint">
 				<hardwareInterface>EffortJointInterface</hardwareInterface>
 			</joint>
-			<actuator name="${name}_arm_4_motor">
+			<actuator name="${name}_4_motor">
 				<hardwareInterface>EffortJointInterface</hardwareInterface>
 				<mechanicalReduction>1</mechanicalReduction>
 			</actuator>
 		</transmission>
-		<transmission name="${name}_arm_5_trans">
+		<transmission name="${name}_5_trans">
 			<type>transmission_interface/SimpleTransmission</type>
-			<joint name="${name}_arm_5_joint">
+			<joint name="${name}_5_joint">
 				<hardwareInterface>EffortJointInterface</hardwareInterface>
 			</joint>
-			<actuator name="${name}_arm_5_motor">
+			<actuator name="${name}_5_motor">
 				<hardwareInterface>EffortJointInterface</hardwareInterface>
 				<mechanicalReduction>1</mechanicalReduction>
 			</actuator>
 		</transmission>
-		<transmission name="${name}_arm_6_trans">
+		<transmission name="${name}_6_trans">
 			<type>transmission_interface/SimpleTransmission</type>
-			<joint name="${name}_arm_6_joint">
+			<joint name="${name}_6_joint">
 				<hardwareInterface>EffortJointInterface</hardwareInterface>
 			</joint>
-			<actuator name="${name}_arm_6_motor">
+			<actuator name="${name}_6_motor">
 				<hardwareInterface>EffortJointInterface</hardwareInterface>
 				<mechanicalReduction>1</mechanicalReduction>

File: ros/kuka_lwr/lwr_description/model/kuka_lwr.urdf.xacro (robot description, xacro)
@@ -15,11 +15,11 @@
 	<xacro:macro name="kuka_lwr" params="parent name *origin">
 	<!-- First (shoulder) element of the arm. Fixed to its parent. -->
-	<joint name="${parent}_${name}_arm_base_joint" type="fixed">
+	<joint name="${parent}_${name}_base_joint" type="fixed">
 		<insert_block name="origin"/>
 		<origin xyz="0 0 0" rpy="0 0 0"/>
 		<parent link="${parent}"/>
-		<child link="${name}_arm_base_link"/>
-	</joint>
-	<link name="${name}_arm_base_link">
+		<child link="${name}_base_link"/>
+	</joint>
+	<link name="${name}_base_link">
 		<inertial>
 			<mass value="${base_mass}"/>
@@ -43,5 +43,5 @@
 	</link>
 	<!-- Second segment of the arm. Joint along z-axis -->
-	<joint name="${name}_arm_0_joint" type="revolute">
+	<joint name="${name}_0_joint" type="revolute">
 		<origin xyz="0 0 0.11" rpy="0 0 0"/>
 		<axis xyz="0 0 1"/>
@@ -49,8 +49,8 @@
 		<safety_controller soft_lower_limit="${-168 * M_PI / 180}" soft_upper_limit="${168 * M_PI / 180}" k_position="30" k_velocity="30"/>
 		<dynamics damping="1.0"/>
-		<parent link="${name}_arm_base_link"/>
-		<child link="${name}_arm_1_link"/>
-	</joint>
-	<link name="${name}_arm_1_link">
+		<parent link="${name}_base_link"/>
+		<child link="${name}_1_link"/>
+	</joint>
+	<link name="${name}_1_link">
 		<inertial>
 			<mass value="${link_mass}"/>
@@ -86,5 +86,5 @@
 	</link>
 	<!-- Third segment of the arm. Joint along y-axis -->
-	<joint name="${name}_arm_1_joint" type="revolute">
+	<joint name="${name}_1_joint" type="revolute">
 		<origin xyz="0 0 0.2005" rpy="0 0 0"/>
 		<axis xyz="0 -1 0"/>
@@ -93,8 +93,8 @@
 		<safety_controller soft_lower_limit="${-118 * M_PI / 180}" soft_upper_limit="${118 * M_PI / 180}" k_position="30" k_velocity="30"/>
 		<dynamics damping="1.0"/>
-		<parent link="${name}_arm_1_link"/>
-		<child link="${name}_arm_2_link"/>
-	</joint>
-	<link name="${name}_arm_2_link">
+		<parent link="${name}_1_link"/>
+		<child link="${name}_2_link"/>
+	</joint>
+	<link name="${name}_2_link">
 		<inertial>
 			<mass value="${link_mass}"/>
@@ -130,5 +130,5 @@
 	</link>
 	<!-- Fourth element of the arm. z-axis -->
-	<joint name="${name}_arm_2_joint" type="revolute">
+	<joint name="${name}_2_joint" type="revolute">
 		<origin xyz="0 0 0.20" rpy="0 0 0"/>
 		<axis xyz="0 0 1"/>
@@ -136,8 +136,8 @@
 		<safety_controller soft_lower_limit="${-168 * M_PI / 180}" soft_upper_limit="${168 * M_PI / 180}" k_position="30" k_velocity="30"/>
 		<dynamics damping="1.0"/>
-		<parent link="${name}_arm_2_link"/>
-		<child link="${name}_arm_3_link"/>
-	</joint>
-	<link name="${name}_arm_3_link">
+		<parent link="${name}_2_link"/>
+		<child link="${name}_3_link"/>
+	</joint>
+	<link name="${name}_3_link">
 		<inertial>
 			<mass value="${link_mass}"/>
@@ -173,5 +173,5 @@
 	</link>
 	<!-- fifth element of the arm. x-axis -->
-	<joint name="${name}_arm_3_joint" type="revolute">
+	<joint name="${name}_3_joint" type="revolute">
 		<origin xyz="0 0 0.20" rpy="0 0 0"/>
 		<axis xyz="0 1 0"/>
@@ -179,8 +179,8 @@
 			<safety_controller soft_lower_limit="${-118 * M_PI / 180}" soft_upper_limit="${118 * M_PI / 180}" k_position="30" k_velocity="30"/>
 		<dynamics damping="1.0"/>
-		<parent link="${name}_arm_3_link"/>
-		<child link="${name}_arm_4_link"/>
-	</joint>
-	<link name="${name}_arm_4_link">
+		<parent link="${name}_3_link"/>
+		<child link="${name}_4_link"/>
+	</joint>
+	<link name="${name}_4_link">
 		<inertial>
 			<mass value="${link_mass}"/>
@@ -216,5 +216,5 @@
 	</link>
 	<!-- Sixth element of the arm. z-axis -->
-	<joint name="${name}_arm_4_joint" type="revolute">
+	<joint name="${name}_4_joint" type="revolute">
 		<origin xyz="0 0 0.20" rpy="0 0 0"/>
 		<axis xyz="0 0 1"/>
@@ -222,8 +222,8 @@
 		<safety_controller soft_lower_limit="${-168 * M_PI / 180}" soft_upper_limit="${168 * M_PI / 180}" k_position="30" k_velocity="30"/>
 		<dynamics damping="1.0"/>
-		<parent link="${name}_arm_4_link"/>
-		<child link="${name}_arm_5_link"/>
-	</joint>
-	<link name="${name}_arm_5_link">
+		<parent link="${name}_4_link"/>
+		<child link="${name}_5_link"/>
+	</joint>
+	<link name="${name}_5_link">
 		<inertial>
 			<mass value="${link_mass}"/>
@@ -233,5 +233,5 @@
 		<visual>
 			<origin xyz="0 0 -0.008" rpy="0 0 ${M_PI}"/>
-			<geometry name="${name}_arm_5_geom">
+			<geometry name="${name}_5_geom">
 				<mesh filename="package://lwr_description/meshes/link_5.STL"/>
 			</geometry>
@@ -259,5 +259,5 @@
 	</link>
 	<!-- Seventh element of the arm. z-axis -->
-	<joint name="${name}_arm_5_joint" type="revolute">
+	<joint name="${name}_5_joint" type="revolute">
 		<origin xyz="0 0 0.19" rpy="0 0 0"/>
 		<axis xyz="0 -1 0"/>
@@ -265,8 +265,8 @@
 		<safety_controller soft_lower_limit="${-118 * M_PI / 180}" soft_upper_limit="${118 * M_PI / 180}" k_position="30" k_velocity="30"/>
 		<dynamics damping="1.0"/>
-		<parent link="${name}_arm_5_link"/>
-		<child link="${name}_arm_6_link"/>
-	</joint>
-	<link name="${name}_arm_6_link">
+		<parent link="${name}_5_link"/>
+		<child link="${name}_6_link"/>
+	</joint>
+	<link name="${name}_6_link">
 		<inertial>
 			<mass value="0.2"/>
@@ -289,5 +289,5 @@
 	</link>
 	<!-- Eighth element of the arm. z-axis -->
-	<joint name="${name}_arm_6_joint" type="revolute">
+	<joint name="${name}_6_joint" type="revolute">
 		<origin xyz="0 0 0.078" rpy="0 0 0"/>
 		<axis xyz="0 0 1"/>
@@ -295,8 +295,8 @@
 		<safety_controller soft_lower_limit="${-168 * M_PI / 180}" soft_upper_limit="${168 * M_PI / 180}" k_position="30" k_velocity="30"/>
 		<dynamics damping="1.0"/>
-		<parent link="${name}_arm_6_link"/>
-		<child link="${name}_arm_7_link"/>
-	</joint>
-	<link name="${name}_arm_7_link">
+		<parent link="${name}_6_link"/>
+		<child link="${name}_7_link"/>
+	</joint>
+	<link name="${name}_7_link">
 		<inertial>
 			<mass value="0.2"/>
