Commit message: update controller gains and moveit package

File: ros/kuka_lwr/lwr_description/model/kuka_lwr.urdf.xacro (robot description, xacro)
@@ -11,5 +11,5 @@
 	<xacro:property name="base_mass" value="2.0"/>
 	<xacro:property name="link_mass" value="2.0"/>
-	<xacro:property name="velocity_scale" value="1"/>
+	<xacro:property name="velocity_scale" value="3"/>
 	<!-- URDF model /-->
 	<xacro:macro name="kuka_lwr" params="parent name *origin">
@@ -48,5 +48,5 @@
 		<limit lower="${-170 * M_PI / 180}" upper="${170 * M_PI / 180}" effort="204" velocity="${velocity_scale * 110 * M_PI / 180}" />
 		<safety_controller soft_lower_limit="${-168 * M_PI / 180}" soft_upper_limit="${168 * M_PI / 180}" k_position="30" k_velocity="30"/>
-		<dynamics damping="1.0"/>
+		<dynamics friction="10.0" damping="1.0"/>
 		<parent link="${name}_base_link"/>
 		<child link="${name}_1_link"/>
@@ -92,5 +92,5 @@
 			 effort="306" velocity="${velocity_scale * 110 * M_PI / 180}" />
 		<safety_controller soft_lower_limit="${-118 * M_PI / 180}" soft_upper_limit="${118 * M_PI / 180}" k_position="30" k_velocity="30"/>
-		<dynamics damping="1.0"/>
+		<dynamics friction="10.0" damping="1.0"/>
 		<parent link="${name}_1_link"/>
 		<child link="${name}_2_link"/>
@@ -135,5 +135,5 @@
 		<limit lower="${-170 * M_PI / 180}" upper="${170 * M_PI / 180}" effort="204" velocity="${velocity_scale * 130 * M_PI / 180}" />
 		<safety_controller soft_lower_limit="${-168 * M_PI / 180}" soft_upper_limit="${168 * M_PI / 180}" k_position="30" k_velocity="30"/>
-		<dynamics damping="1.0"/>
+		<dynamics friction="10.0" damping="1.0"/>
 		<parent link="${name}_2_link"/>
 		<child link="${name}_3_link"/>
@@ -178,5 +178,5 @@
 		<limit lower="${-120 * M_PI / 180}" upper="${120 * M_PI / 180}" effort="306" velocity="${velocity_scale * 130 * M_PI / 180}" />
 			<safety_controller soft_lower_limit="${-118 * M_PI / 180}" soft_upper_limit="${118 * M_PI / 180}" k_position="30" k_velocity="30"/>
-		<dynamics damping="1.0"/>
+		<dynamics friction="10.0" damping="1.0"/>
 		<parent link="${name}_3_link"/>
 		<child link="${name}_4_link"/>
@@ -221,5 +221,5 @@
 		<limit lower="${-170 * M_PI / 180}" upper="${170 * M_PI / 180}" effort="204" velocity="${velocity_scale * 130 * M_PI / 180}" />
 		<safety_controller soft_lower_limit="${-168 * M_PI / 180}" soft_upper_limit="${168 * M_PI / 180}" k_position="30" k_velocity="30"/>
-		<dynamics damping="1.0"/>
+		<dynamics friction="10.0" damping="1.0"/>
 		<parent link="${name}_4_link"/>
 		<child link="${name}_5_link"/>
@@ -264,5 +264,5 @@
 		<limit lower="${-120 * M_PI / 180}" upper="${120 * M_PI / 180}" effort="306" velocity="${velocity_scale * 180 * M_PI / 180}" />
 		<safety_controller soft_lower_limit="${-118 * M_PI / 180}" soft_upper_limit="${118 * M_PI / 180}" k_position="30" k_velocity="30"/>
-		<dynamics damping="1.0"/>
+		<dynamics friction="10.0" damping="1.0"/>
 		<parent link="${name}_5_link"/>
 		<child link="${name}_6_link"/>
@@ -294,5 +294,5 @@
 		<limit lower="${-170 * M_PI / 180}" upper="${170 * M_PI / 180}" effort="204" velocity="${velocity_scale * 180 * M_PI / 180}" />
 		<safety_controller soft_lower_limit="${-168 * M_PI / 180}" soft_upper_limit="${168 * M_PI / 180}" k_position="30" k_velocity="30"/>
-		<dynamics damping="1.0"/>
+		<dynamics friction="10.0" damping="1.0"/>
 		<parent link="${name}_6_link"/>
 		<child link="${name}_7_link"/>
