Commit message: [lwr_description] Updating URDF with values from the kuka manuals.

File: lwr_description/model/kuka_lwr.urdf.xacro (robot description, xacro)
@@ -11,5 +11,6 @@
 	<xacro:property name="base_mass" value="2.0"/>
 	<xacro:property name="link_mass" value="2.0"/>
-	<xacro:property name="velocity_scale" value="3"/>
+	<xacro:property name="velocity_scale" value="1"/>
+	<xacro:property name="effort_scale" value="1"/>
 	<!-- URDF model /-->
 	<xacro:macro name="kuka_lwr" params="parent name *origin">
@@ -46,6 +47,6 @@
 		<origin xyz="0 0 0.11" rpy="0 0 0"/>
 		<axis xyz="0 0 1"/>
-		<limit lower="${-170 * M_PI / 180}" upper="${170 * M_PI / 180}" effort="204" velocity="${velocity_scale * 110 * M_PI / 180}" />
-		<safety_controller soft_lower_limit="${-168 * M_PI / 180}" soft_upper_limit="${168 * M_PI / 180}" k_position="30" k_velocity="30"/>
+		<limit lower="${-170 * M_PI / 180}" upper="${170 * M_PI / 180}" effort="176" velocity="${velocity_scale * 110 * M_PI / 180}" />
+		<safety_controller soft_lower_limit="${-160 * M_PI / 180}" soft_upper_limit="${160 * M_PI / 180}" k_position="30" k_velocity="30"/>
 		<dynamics friction="10.0" damping="1.0"/>
 		<parent link="${name}_base_link"/>
@@ -89,7 +90,6 @@
 		<origin xyz="0 0 0.2005" rpy="0 0 0"/>
 		<axis xyz="0 -1 0"/>
-		<limit lower="${-120 * M_PI / 180}" upper="${120 * M_PI / 180}"
-			 effort="306" velocity="${velocity_scale * 110 * M_PI / 180}" />
-		<safety_controller soft_lower_limit="${-118 * M_PI / 180}" soft_upper_limit="${118 * M_PI / 180}" k_position="30" k_velocity="30"/>
+		<limit lower="${-120 * M_PI / 180}" upper="${120 * M_PI / 180}" effort="176" velocity="${velocity_scale * 110 * M_PI / 180}" />
+		<safety_controller soft_lower_limit="${-110 * M_PI / 180}" soft_upper_limit="${110 * M_PI / 180}" k_position="30" k_velocity="30"/>
 		<dynamics friction="10.0" damping="1.0"/>
 		<parent link="${name}_1_link"/>
@@ -133,6 +133,6 @@
 		<origin xyz="0 0 0.20" rpy="0 0 0"/>
 		<axis xyz="0 0 1"/>
-		<limit lower="${-170 * M_PI / 180}" upper="${170 * M_PI / 180}" effort="204" velocity="${velocity_scale * 130 * M_PI / 180}" />
-		<safety_controller soft_lower_limit="${-168 * M_PI / 180}" soft_upper_limit="${168 * M_PI / 180}" k_position="30" k_velocity="30"/>
+		<limit lower="${-170 * M_PI / 180}" upper="${170 * M_PI / 180}" effort="100" velocity="${velocity_scale * 128 * M_PI / 180}" />
+		<safety_controller soft_lower_limit="${-160 * M_PI / 180}" soft_upper_limit="${160 * M_PI / 180}" k_position="30" k_velocity="30"/>
 		<dynamics friction="10.0" damping="1.0"/>
 		<parent link="${name}_2_link"/>
@@ -176,6 +176,6 @@
 		<origin xyz="0 0 0.20" rpy="0 0 0"/>
 		<axis xyz="0 1 0"/>
-		<limit lower="${-120 * M_PI / 180}" upper="${120 * M_PI / 180}" effort="306" velocity="${velocity_scale * 130 * M_PI / 180}" />
-			<safety_controller soft_lower_limit="${-118 * M_PI / 180}" soft_upper_limit="${118 * M_PI / 180}" k_position="30" k_velocity="30"/>
+		<limit lower="${-120 * M_PI / 180}" upper="${120 * M_PI / 180}" effort="100" velocity="${velocity_scale * 128 * M_PI / 180}" />
+			<safety_controller soft_lower_limit="${-110 * M_PI / 180}" soft_upper_limit="${110 * M_PI / 180}" k_position="30" k_velocity="30"/>
 		<dynamics friction="10.0" damping="1.0"/>
 		<parent link="${name}_3_link"/>
@@ -219,6 +219,6 @@
 		<origin xyz="0 0 0.20" rpy="0 0 0"/>
 		<axis xyz="0 0 1"/>
-		<limit lower="${-170 * M_PI / 180}" upper="${170 * M_PI / 180}" effort="204" velocity="${velocity_scale * 130 * M_PI / 180}" />
-		<safety_controller soft_lower_limit="${-168 * M_PI / 180}" soft_upper_limit="${168 * M_PI / 180}" k_position="30" k_velocity="30"/>
+		<limit lower="${-170 * M_PI / 180}" upper="${170 * M_PI / 180}" effort="100" velocity="${velocity_scale * 204 * M_PI / 180}" />
+		<safety_controller soft_lower_limit="${-160 * M_PI / 180}" soft_upper_limit="${160 * M_PI / 180}" k_position="30" k_velocity="30"/>
 		<dynamics friction="10.0" damping="1.0"/>
 		<parent link="${name}_4_link"/>
@@ -262,6 +262,6 @@
 		<origin xyz="0 0 0.19" rpy="0 0 0"/>
 		<axis xyz="0 -1 0"/>
-		<limit lower="${-120 * M_PI / 180}" upper="${120 * M_PI / 180}" effort="306" velocity="${velocity_scale * 180 * M_PI / 180}" />
-		<safety_controller soft_lower_limit="${-118 * M_PI / 180}" soft_upper_limit="${118 * M_PI / 180}" k_position="30" k_velocity="30"/>
+		<limit lower="${-120 * M_PI / 180}" upper="${120 * M_PI / 180}" effort="38" velocity="${velocity_scale * 184 * M_PI / 180}" />
+		<safety_controller soft_lower_limit="${-110 * M_PI / 180}" soft_upper_limit="${110 * M_PI / 180}" k_position="30" k_velocity="30"/>
 		<dynamics friction="10.0" damping="1.0"/>
 		<parent link="${name}_5_link"/>
@@ -292,6 +292,6 @@
 		<origin xyz="0 0 0.078" rpy="0 0 0"/>
 		<axis xyz="0 0 1"/>
-		<limit lower="${-170 * M_PI / 180}" upper="${170 * M_PI / 180}" effort="204" velocity="${velocity_scale * 180 * M_PI / 180}" />
-		<safety_controller soft_lower_limit="${-168 * M_PI / 180}" soft_upper_limit="${168 * M_PI / 180}" k_position="30" k_velocity="30"/>
+		<limit lower="${-170 * M_PI / 180}" upper="${170 * M_PI / 180}" effort="38" velocity="${velocity_scale * 184 * M_PI / 180}" />
+		<safety_controller soft_lower_limit="${-160 * M_PI / 180}" soft_upper_limit="${160 * M_PI / 180}" k_position="30" k_velocity="30"/>
 		<dynamics friction="10.0" damping="1.0"/>
 		<parent link="${name}_6_link"/>

Commit message: Updated URDF link mass

File: lwr_description/model/kuka_lwr.urdf.xacro (robot description, xacro)
@@ -10,5 +10,7 @@
 	<!-- properties /-->
 	<xacro:property name="base_mass" value="2.0"/>
-	<xacro:property name="link_mass" value="2.0"/>
+	<xacro:property name="link_mass" value="2.35"/>
+    <xacro:property name="wrist_mass" value="1.1"/>
+    <xacro:property name="tip_mass" value="0.25"/>
 	<xacro:property name="velocity_scale" value="1"/>
 	<xacro:property name="effort_scale" value="1"/>
@@ -309,7 +311,7 @@
 		<link name="${name}_6_link">
 			<inertial>
-				<mass value="0.2"/>
+				<mass value="${wrist_mass}"/>
 				<origin rpy="0 0 0" xyz="0 0 0.0625"/>
-				<cuboid_inertia_def length="0.125" width="0.125" height="0.125" mass="0.2"/>
+				<cuboid_inertia_def length="0.125" width="0.125" height="0.125" mass="${wrist_mass}"/>
 			</inertial>
 			<visual>
@@ -346,7 +348,7 @@
 		<link name="${name}_7_link">
 			<inertial>
-				<mass value="0.2"/>
+				<mass value="${tip_mass}"/>
 				<origin xyz="0 0 0"/>
-				<cuboid_inertia_def length="1" width="1" height="1" mass="0.2"/>
+				<cuboid_inertia_def length="0.1" width="0.1" height="0.1" mass="${tip_mass}"/>
 			</inertial>
 			<visual>

Commit message: Updated URDF link mass

File: lwr_description/model/kuka_lwr.urdf.xacro (robot description, xacro)
@@ -10,5 +10,7 @@
 	<!-- properties /-->
 	<xacro:property name="base_mass" value="2.0"/>
-	<xacro:property name="link_mass" value="2.0"/>
+	<xacro:property name="link_mass" value="2.35"/>
+    <xacro:property name="wrist_mass" value="1.1"/>
+    <xacro:property name="tip_mass" value="0.25"/>
 	<xacro:property name="velocity_scale" value="1"/>
 	<xacro:property name="effort_scale" value="1"/>
@@ -315,7 +317,7 @@
 	<link name="${name}_6_link">
 		<inertial>
-			<mass value="0.2"/>
+			<mass value="${wrist_mass}"/>
 			<origin rpy="0 0 0" xyz="0 0 0.0625"/>
-			<cuboid_inertia_def length="0.125" width="0.125" height="0.125" mass="0.2"/>
+			<cuboid_inertia_def length="0.125" width="0.125" height="0.125" mass="${wrist_mass}"/>
 		</inertial>
 		<visual>
@@ -352,7 +354,7 @@
 	<link name="${name}_7_link">
 		<inertial>
-			<mass value="0.2"/>
+			<mass value="${tip_mass}"/>
 			<origin xyz="0 0 0"/>
-			<cuboid_inertia_def length="1" width="1" height="1" mass="0.2"/>
+			<cuboid_inertia_def length="0.1" width="0.1" height="0.1" mass="${tip_mass}"/>
 		</inertial>
 		<visual>
