Commit message: [lwr_hw_sim] Initial import of the lwr_hw_sim package that implements the default lwr sim interface that emulates the joint impedance control strategy. [lwr_description] URDF/xacro model updated to use this interface in simulation, and [lwr_launch] Default launch is in simulation with joint position trajectory. Close #3

File: lwr_description/model/kuka_lwr.gazebo.xacro (robot description, xacro)
@@ -5,4 +5,6 @@
 			<plugin name="gazebo_ros_control" filename="libgazebo_ros_control.so">
 				<robotNamespace>${name}</robotNamespace>
+				<!-- A default KUKA LWR 4+ simulation interface that emulates the joint impedance control strategy -->
+				<robotSimType>gazebo_ros_control/DefaultLWRHWSim</robotSimType>
 			</plugin>
 		</gazebo>

File: lwr_description/robot/lwr_on_box.urdf.xacro (robot description, xacro)
@@ -3,9 +3,4 @@
 	<xacro:include filename="$(find lwr_description)/model/kuka_lwr.urdf.xacro"/>
 	<link name="world">
-		<inertial>
-			<mass value="50.0"/>
-			<com xyz="0 0 0"/>
-			<inertia  ixx="0.01" ixy="0.00"  ixz="0.00" iyy="0.01" iyz="0.00" izz="0.01" />
-		</inertial>
 		<visual>
 			<origin xyz="0 0 0.50" rpy="0 0 0"/>

Commit message: Changes to reflect the changes in the lwr_hw package. Now, URDF uses interfaces from there.
Now there are joint stiffness that are used to control in position/trajectory the stiffness of the real/sim joints.

File: lwr_description/model/kuka_lwr.gazebo.xacro (robot description, xacro)
@@ -3,8 +3,8 @@
 	<xacro:macro name="kuka_lwr_gazebo" params="name">
 		<gazebo>
-			<plugin name="gazebo_ros_control" filename="libgazebo_ros_control.so">
+			<plugin name="lwr_hw" filename="liblwr_hw_sim_plugin.so">
 				<robotNamespace>${name}</robotNamespace>
 				<!-- A default KUKA LWR 4+ simulation interface that emulates the joint impedance control strategy -->
-				<robotSimType>gazebo_ros_control/DefaultLWRHWSim</robotSimType>
+				<robotSimType>lwr_hw/DefaultLWRHWsim</robotSimType>
 			</plugin>
 		</gazebo>

File: lwr_description/model/kuka_lwr.transmission.xacro (robot description, xacro)
@@ -6,8 +6,7 @@
 			<type>transmission_interface/SimpleTransmission</type>
 			<joint name="${name}_0_joint">
-				<hardwareInterface>EffortJointInterface</hardwareInterface>
+				<hardwareInterface>PositionJointInterface</hardwareInterface>
 			</joint>
 			<actuator name="${name}_0_motor">
-				<hardwareInterface>EffortJointInterface</hardwareInterface>
 				<mechanicalReduction>1</mechanicalReduction>
 			</actuator>
@@ -17,8 +16,7 @@
 			<type>transmission_interface/SimpleTransmission</type>
 			<joint name="${name}_1_joint">
-				<hardwareInterface>EffortJointInterface</hardwareInterface>
+				<hardwareInterface>PositionJointInterface</hardwareInterface>
 			</joint>
 			<actuator name="${name}_1_motor">
-				<hardwareInterface>EffortJointInterface</hardwareInterface>
 				<mechanicalReduction>1</mechanicalReduction>
 			</actuator>
@@ -28,8 +26,7 @@
 			<type>transmission_interface/SimpleTransmission</type>
 			<joint name="${name}_2_joint">
-				<hardwareInterface>EffortJointInterface</hardwareInterface>
+				<hardwareInterface>PositionJointInterface</hardwareInterface>
 			</joint>
 			<actuator name="${name}_2_motor">
-				<hardwareInterface>EffortJointInterface</hardwareInterface>
 				<mechanicalReduction>1</mechanicalReduction>
 			</actuator>
@@ -39,8 +36,7 @@
 			<type>transmission_interface/SimpleTransmission</type>
 			<joint name="${name}_3_joint">
-				<hardwareInterface>EffortJointInterface</hardwareInterface>
+				<hardwareInterface>PositionJointInterface</hardwareInterface>
 			</joint>
 			<actuator name="${name}_3_motor">
-				<hardwareInterface>EffortJointInterface</hardwareInterface>
 				<mechanicalReduction>1</mechanicalReduction>
 			</actuator>
@@ -50,8 +46,7 @@
 			<type>transmission_interface/SimpleTransmission</type>
 			<joint name="${name}_4_joint">
-				<hardwareInterface>EffortJointInterface</hardwareInterface>
+				<hardwareInterface>PositionJointInterface</hardwareInterface>
 			</joint>
 			<actuator name="${name}_4_motor">
-				<hardwareInterface>EffortJointInterface</hardwareInterface>
 				<mechanicalReduction>1</mechanicalReduction>
 			</actuator>
@@ -61,8 +56,7 @@
 			<type>transmission_interface/SimpleTransmission</type>
 			<joint name="${name}_5_joint">
-				<hardwareInterface>EffortJointInterface</hardwareInterface>
+				<hardwareInterface>PositionJointInterface</hardwareInterface>
 			</joint>
 			<actuator name="${name}_5_motor">
-				<hardwareInterface>EffortJointInterface</hardwareInterface>
 				<mechanicalReduction>1</mechanicalReduction>
 			</actuator>
@@ -72,11 +66,80 @@
 			<type>transmission_interface/SimpleTransmission</type>
 			<joint name="${name}_6_joint">
-				<hardwareInterface>EffortJointInterface</hardwareInterface>
+				<hardwareInterface>PositionJointInterface</hardwareInterface>
 			</joint>
 			<actuator name="${name}_6_motor">
-				<hardwareInterface>EffortJointInterface</hardwareInterface>
 				<mechanicalReduction>1</mechanicalReduction>
 			</actuator>
 		</transmission>
+		<!-- <transmission name="${name}_0_trans_stiff">
+			<robotNamespace>${name}</robotNamespace>
+			<type>transmission_interface/SimpleTransmission</type>
+			<joint name="${name}_0_joint_stiffness">
+				<hardwareInterface>PositionJointInterface</hardwareInterface>
+			</joint>
+			<actuator name="${name}_0_position">
+				<mechanicalReduction>1</mechanicalReduction>
+			</actuator>
+		</transmission>
+		<transmission name="${name}_1_trans_stiff">
+			<robotNamespace>${name}</robotNamespace>
+			<type>transmission_interface/SimpleTransmission</type>
+			<joint name="${name}_1_joint_stiffness">
+				<hardwareInterface>PositionJointInterface</hardwareInterface>
+			</joint>
+			<actuator name="${name}_1_position">
+				<mechanicalReduction>1</mechanicalReduction>
+			</actuator>
+		</transmission>
+		<transmission name="${name}_2_trans_stiff">
+			<robotNamespace>${name}</robotNamespace>
+			<type>transmission_interface/SimpleTransmission</type>
+			<joint name="${name}_2_joint_stiffness">
+				<hardwareInterface>PositionJointInterface</hardwareInterface>
+			</joint>
+			<actuator name="${name}_2_position">
+				<mechanicalReduction>1</mechanicalReduction>
+			</actuator>
+		</transmission>
+		<transmission name="${name}_3_trans_stiff">
+			<robotNamespace>${name}</robotNamespace>
+			<type>transmission_interface/SimpleTransmission</type>
+			<joint name="${name}_3_joint_stiffness">
+				<hardwareInterface>PositionJointInterface</hardwareInterface>
+			</joint>
+			<actuator name="${name}_3_position">
+				<mechanicalReduction>1</mechanicalReduction>
+			</actuator>
+		</transmission>
+		<transmission name="${name}_4_trans_stiff">
+			<robotNamespace>${name}</robotNamespace>
+			<type>transmission_interface/SimpleTransmission</type>
+			<joint name="${name}_4_joint_stiffness">
+				<hardwareInterface>PositionJointInterface</hardwareInterface>
+			</joint>
+			<actuator name="${name}_4_position">
+				<mechanicalReduction>1</mechanicalReduction>
+			</actuator>
+		</transmission>
+		<transmission name="${name}_5_trans_stiff">
+			<robotNamespace>${name}</robotNamespace>
+			<type>transmission_interface/SimpleTransmission</type>
+			<joint name="${name}_5_joint_stiffness">
+				<hardwareInterface>PositionJointInterface</hardwareInterface>
+			</joint>
+			<actuator name="${name}_5_position">
+				<mechanicalReduction>1</mechanicalReduction>
+			</actuator>
+		</transmission>
+		<transmission name="${name}_6_trans_stiff">
+			<robotNamespace>${name}</robotNamespace>
+			<type>transmission_interface/SimpleTransmission</type>
+			<joint name="${name}_6_joint_stiffness">
+				<hardwareInterface>PositionJointInterface</hardwareInterface>
+			</joint>
+			<actuator name="${name}_6_position">
+				<mechanicalReduction>1</mechanicalReduction>
+			</actuator>
+		</transmission> -->
 	</xacro:macro>
 </robot>

File: lwr_description/model/kuka_lwr.urdf.xacro (robot description, xacro)
@@ -13,4 +13,7 @@
 	<xacro:property name="velocity_scale" value="1"/>
 	<xacro:property name="effort_scale" value="1"/>
+	<xacro:property name="max_stiffness" value="5000"/>
+	<xacro:property name="min_stiffness" value="0"/>
+	<xacro:property name="rate_stiffness" value="20000"/> <!-- reflex to stiffness -->
 	<!-- URDF model /-->
 	<xacro:macro name="kuka_lwr" params="parent name *origin">
@@ -53,4 +56,12 @@
 		<child link="${name}_1_link"/>
 	</joint>
+	<joint name="${name}_0_joint_stiffness" type="revolute">
+		<axis xyz="0 0 1"/>
+		<limit lower="${min_stiffness}" upper="${max_stiffness}" effort="0" velocity="${rate_stiffness}" />
+		<safety_controller soft_lower_limit="${min_stiffness}" soft_upper_limit="${max_stiffness}" k_position="30" k_velocity="30"/>
+		<parent link="${name}_base_link"/>
+		<child link="${name}_1_link_dummy"/>
+	</joint>
+	<link name="${name}_1_link_dummy"/>
 	<link name="${name}_1_link">
 		<inertial>
@@ -96,4 +107,12 @@
 		<child link="${name}_2_link"/>
 	</joint>
+	<joint name="${name}_1_joint_stiffness" type="revolute">
+		<axis xyz="0 0 1"/>
+		<limit lower="${min_stiffness}" upper="${max_stiffness}" effort="0" velocity="${rate_stiffness}" />
+		<safety_controller soft_lower_limit="${min_stiffness}" soft_upper_limit="${max_stiffness}" k_position="30" k_velocity="30"/>
+		<parent link="${name}_1_link"/>
+		<child link="${name}_2_link_dummy"/>
+	</joint>
+	<link name="${name}_2_link_dummy"/>
 	<link name="${name}_2_link">
 		<inertial>
@@ -139,4 +158,12 @@
 		<child link="${name}_3_link"/>
 	</joint>
+	<joint name="${name}_2_joint_stiffness" type="revolute">
+		<axis xyz="0 0 1"/>
+		<limit lower="${min_stiffness}" upper="${max_stiffness}" effort="0" velocity="${rate_stiffness}" />
+		<safety_controller soft_lower_limit="${min_stiffness}" soft_upper_limit="${max_stiffness}" k_position="30" k_velocity="30"/>
+		<parent link="${name}_2_link"/>
+		<child link="${name}_3_link_dummy"/>
+	</joint>
+	<link name="${name}_3_link_dummy"/>
 	<link name="${name}_3_link">
 		<inertial>
@@ -182,4 +209,12 @@
 		<child link="${name}_4_link"/>
 	</joint>
+	<joint name="${name}_3_joint_stiffness" type="revolute">
+		<axis xyz="0 0 1"/>
+		<limit lower="${min_stiffness}" upper="${max_stiffness}" effort="0" velocity="${rate_stiffness}" />
+		<safety_controller soft_lower_limit="${min_stiffness}" soft_upper_limit="${max_stiffness}" k_position="30" k_velocity="30"/>
+		<parent link="${name}_3_link"/>
+		<child link="${name}_4_link_dummy"/>
+	</joint>
+	<link name="${name}_4_link_dummy"/>
 	<link name="${name}_4_link">
 		<inertial>
@@ -225,4 +260,12 @@
 		<child link="${name}_5_link"/>
 	</joint>
+	<joint name="${name}_4_joint_stiffness" type="revolute">
+		<axis xyz="0 0 1"/>
+		<limit lower="${min_stiffness}" upper="${max_stiffness}" effort="0" velocity="${rate_stiffness}" />
+		<safety_controller soft_lower_limit="${min_stiffness}" soft_upper_limit="${max_stiffness}" k_position="30" k_velocity="30"/>
+		<parent link="${name}_4_link"/>
+		<child link="${name}_5_link_dummy"/>
+	</joint>
+	<link name="${name}_5_link_dummy"/>
 	<link name="${name}_5_link">
 		<inertial>
@@ -268,4 +311,12 @@
 		<child link="${name}_6_link"/>
 	</joint>
+	<joint name="${name}_5_joint_stiffness" type="revolute">
+		<axis xyz="0 0 1"/>
+		<limit lower="${min_stiffness}" upper="${max_stiffness}" effort="0" velocity="${rate_stiffness}" />
+		<safety_controller soft_lower_limit="${min_stiffness}" soft_upper_limit="${max_stiffness}" k_position="30" k_velocity="30"/>
+		<parent link="${name}_5_link"/>
+		<child link="${name}_6_link_dummy"/>
+	</joint>
+	<link name="${name}_6_link_dummy"/>
 	<link name="${name}_6_link">
 		<inertial>
@@ -298,4 +349,12 @@
 		<child link="${name}_7_link"/>
 	</joint>
+	<joint name="${name}_6_joint_stiffness" type="revolute">
+		<axis xyz="0 0 1"/>
+		<limit lower="${min_stiffness}" upper="${max_stiffness}" effort="0" velocity="${rate_stiffness}" />
+		<safety_controller soft_lower_limit="${min_stiffness}" soft_upper_limit="${max_stiffness}" k_position="30" k_velocity="30"/>
+		<parent link="${name}_6_link"/>
+		<child link="${name}_7_link_dummy"/>
+	</joint>
+	<link name="${name}_7_link_dummy"/>
 	<link name="${name}_7_link">
 		<inertial>

Commit message: Initial work in the update of the lwr_hw package

File: lwr_description/model/kuka_lwr.gazebo.xacro (robot description, xacro)
@@ -5,6 +5,4 @@
 			<plugin name="lwr_hw" filename="liblwr_hw_sim_plugin.so">
 				<robotNamespace>${name}</robotNamespace>
-				<!-- A default KUKA LWR 4+ simulation interface that emulates the joint impedance control strategy -->
-				<robotSimType>lwr_hw/DefaultLWRHWsim</robotSimType>
 			</plugin>
 		</gazebo>

File: lwr_description/model/kuka_lwr.transmission.xacro (robot description, xacro)
@@ -1,4 +1,6 @@
 <?xml version="1.0"?>
 <robot xmlns:xacro="http://ros.org/wiki/xacro">
+	<xacro:property name="Interface10" value="PositionJointInterface"/>
+	<xacro:property name="Interface30" value="EffortJointInterface"/>
 	<xacro:macro name="kuka_lwr_transmission" params="name">
 		<transmission name="${name}_0_trans">
@@ -6,5 +8,6 @@
 			<type>transmission_interface/SimpleTransmission</type>
 			<joint name="${name}_0_joint">
-				<hardwareInterface>PositionJointInterface</hardwareInterface>
+				<hardwareInterface>${Interface10}</hardwareInterface>
+				<hardwareInterface>${Interface30}</hardwareInterface>
 			</joint>
 			<actuator name="${name}_0_motor">
@@ -16,5 +19,6 @@
 			<type>transmission_interface/SimpleTransmission</type>
 			<joint name="${name}_1_joint">
-				<hardwareInterface>PositionJointInterface</hardwareInterface>
+				<hardwareInterface>${Interface10}</hardwareInterface>
+				<hardwareInterface>${Interface30}</hardwareInterface>
 			</joint>
 			<actuator name="${name}_1_motor">
@@ -26,5 +30,6 @@
 			<type>transmission_interface/SimpleTransmission</type>
 			<joint name="${name}_2_joint">
-				<hardwareInterface>PositionJointInterface</hardwareInterface>
+				<hardwareInterface>${Interface10}</hardwareInterface>
+				<hardwareInterface>${Interface30}</hardwareInterface>
 			</joint>
 			<actuator name="${name}_2_motor">
@@ -36,5 +41,6 @@
 			<type>transmission_interface/SimpleTransmission</type>
 			<joint name="${name}_3_joint">
-				<hardwareInterface>PositionJointInterface</hardwareInterface>
+				<hardwareInterface>${Interface10}</hardwareInterface>
+				<hardwareInterface>${Interface30}</hardwareInterface>
 			</joint>
 			<actuator name="${name}_3_motor">
@@ -46,5 +52,6 @@
 			<type>transmission_interface/SimpleTransmission</type>
 			<joint name="${name}_4_joint">
-				<hardwareInterface>PositionJointInterface</hardwareInterface>
+				<hardwareInterface>${Interface10}</hardwareInterface>
+				<hardwareInterface>${Interface30}</hardwareInterface>
 			</joint>
 			<actuator name="${name}_4_motor">
@@ -56,5 +63,6 @@
 			<type>transmission_interface/SimpleTransmission</type>
 			<joint name="${name}_5_joint">
-				<hardwareInterface>PositionJointInterface</hardwareInterface>
+				<hardwareInterface>${Interface10}</hardwareInterface>
+				<hardwareInterface>${Interface30}</hardwareInterface>
 			</joint>
 			<actuator name="${name}_5_motor">
@@ -66,5 +74,6 @@
 			<type>transmission_interface/SimpleTransmission</type>
 			<joint name="${name}_6_joint">
-				<hardwareInterface>PositionJointInterface</hardwareInterface>
+				<hardwareInterface>${Interface10}</hardwareInterface>
+				<hardwareInterface>${Interface30}</hardwareInterface>
 			</joint>
 			<actuator name="${name}_6_motor">
@@ -72,74 +81,4 @@
 			</actuator>
 		</transmission>
-		<!-- <transmission name="${name}_0_trans_stiff">
-			<robotNamespace>${name}</robotNamespace>
-			<type>transmission_interface/SimpleTransmission</type>
-			<joint name="${name}_0_joint_stiffness">
-				<hardwareInterface>PositionJointInterface</hardwareInterface>
-			</joint>
-			<actuator name="${name}_0_position">
-				<mechanicalReduction>1</mechanicalReduction>
-			</actuator>
-		</transmission>
-		<transmission name="${name}_1_trans_stiff">
-			<robotNamespace>${name}</robotNamespace>
-			<type>transmission_interface/SimpleTransmission</type>
-			<joint name="${name}_1_joint_stiffness">
-				<hardwareInterface>PositionJointInterface</hardwareInterface>
-			</joint>
-			<actuator name="${name}_1_position">
-				<mechanicalReduction>1</mechanicalReduction>
-			</actuator>
-		</transmission>
-		<transmission name="${name}_2_trans_stiff">
-			<robotNamespace>${name}</robotNamespace>
-			<type>transmission_interface/SimpleTransmission</type>
-			<joint name="${name}_2_joint_stiffness">
-				<hardwareInterface>PositionJointInterface</hardwareInterface>
-			</joint>
-			<actuator name="${name}_2_position">
-				<mechanicalReduction>1</mechanicalReduction>
-			</actuator>
-		</transmission>
-		<transmission name="${name}_3_trans_stiff">
-			<robotNamespace>${name}</robotNamespace>
-			<type>transmission_interface/SimpleTransmission</type>
-			<joint name="${name}_3_joint_stiffness">
-				<hardwareInterface>PositionJointInterface</hardwareInterface>
-			</joint>
-			<actuator name="${name}_3_position">
-				<mechanicalReduction>1</mechanicalReduction>
-			</actuator>
-		</transmission>
-		<transmission name="${name}_4_trans_stiff">
-			<robotNamespace>${name}</robotNamespace>
-			<type>transmission_interface/SimpleTransmission</type>
-			<joint name="${name}_4_joint_stiffness">
-				<hardwareInterface>PositionJointInterface</hardwareInterface>
-			</joint>
-			<actuator name="${name}_4_position">
-				<mechanicalReduction>1</mechanicalReduction>
-			</actuator>
-		</transmission>
-		<transmission name="${name}_5_trans_stiff">
-			<robotNamespace>${name}</robotNamespace>
-			<type>transmission_interface/SimpleTransmission</type>
-			<joint name="${name}_5_joint_stiffness">
-				<hardwareInterface>PositionJointInterface</hardwareInterface>
-			</joint>
-			<actuator name="${name}_5_position">
-				<mechanicalReduction>1</mechanicalReduction>
-			</actuator>
-		</transmission>
-		<transmission name="${name}_6_trans_stiff">
-			<robotNamespace>${name}</robotNamespace>
-			<type>transmission_interface/SimpleTransmission</type>
-			<joint name="${name}_6_joint_stiffness">
-				<hardwareInterface>PositionJointInterface</hardwareInterface>
-			</joint>
-			<actuator name="${name}_6_position">
-				<mechanicalReduction>1</mechanicalReduction>
-			</actuator>
-		</transmission> -->
 	</xacro:macro>
 </robot>
