Commit message: Fix tab/spaces in kuka_lwr.transmission.xacro

File: lwr_description/model/kuka_lwr.transmission.xacro (robot description, xacro)
@@ -1,7 +1,7 @@
 <?xml version="1.0"?>
 <robot xmlns:xacro="http://ros.org/wiki/xacro">
-    <xacro:macro name="kuka_lwr_transmission" params="name">
-	    <transmission name="${name}_0_trans">
-	    	<robotNamespace>${name}</robotNamespace>
+	<xacro:macro name="kuka_lwr_transmission" params="name">
+		<transmission name="${name}_0_trans">
+			<robotNamespace>${name}</robotNamespace>
 			<type>transmission_interface/SimpleTransmission</type>
 			<joint name="${name}_0_joint">
@@ -12,5 +12,5 @@
 				<mechanicalReduction>1</mechanicalReduction>
 			</actuator>
-	    </transmission>
+		</transmission>
 		<transmission name="${name}_1_trans">
 			<robotNamespace>${name}</robotNamespace>

Commit message: [lwr_description] The names match the kuka names. Last change to release v1.0.0

File: lwr_description/model/kuka_lwr.transmission.xacro (robot description, xacro)
@@ -4,71 +4,71 @@
 	<xacro:property name="Interface30" value="EffortJointInterface"/>
 	<xacro:macro name="kuka_lwr_transmission" params="name">
-		<transmission name="${name}_0_trans">
+		<transmission name="${name}_a1_trans">
 			<type>transmission_interface/SimpleTransmission</type>
-			<joint name="${name}_0_joint">
+			<joint name="${name}_a1_joint">
 				<hardwareInterface>${Interface10}</hardwareInterface>
 				<hardwareInterface>${Interface30}</hardwareInterface>
 			</joint>
-			<actuator name="${name}_0_motor">
+			<actuator name="${name}_a1_motor">
 				<mechanicalReduction>1</mechanicalReduction>
 			</actuator>
 		</transmission>
-		<transmission name="${name}_1_trans">
+		<transmission name="${name}_a2_trans">
 			<type>transmission_interface/SimpleTransmission</type>
-			<joint name="${name}_1_joint">
+			<joint name="${name}_a2_joint">
 				<hardwareInterface>${Interface10}</hardwareInterface>
 				<hardwareInterface>${Interface30}</hardwareInterface>
 			</joint>
-			<actuator name="${name}_1_motor">
+			<actuator name="${name}_a2_motor">
 				<mechanicalReduction>1</mechanicalReduction>
 			</actuator>
 		</transmission>
-		<transmission name="${name}_2_trans">
+		<transmission name="${name}_e1_trans">
 			<type>transmission_interface/SimpleTransmission</type>
-			<joint name="${name}_2_joint">
+			<joint name="${name}_e1_joint">
 				<hardwareInterface>${Interface10}</hardwareInterface>
 				<hardwareInterface>${Interface30}</hardwareInterface>
 			</joint>
-			<actuator name="${name}_2_motor">
+			<actuator name="${name}_e1_motor">
 				<mechanicalReduction>1</mechanicalReduction>
 			</actuator>
 		</transmission>
-		<transmission name="${name}_3_trans">
+		<transmission name="${name}_a3_trans">
 			<type>transmission_interface/SimpleTransmission</type>
-			<joint name="${name}_3_joint">
+			<joint name="${name}_a3_joint">
 				<hardwareInterface>${Interface10}</hardwareInterface>
 				<hardwareInterface>${Interface30}</hardwareInterface>
 			</joint>
-			<actuator name="${name}_3_motor">
+			<actuator name="${name}_a3_motor">
 				<mechanicalReduction>1</mechanicalReduction>
 			</actuator>
 		</transmission>
-		<transmission name="${name}_4_trans">
+		<transmission name="${name}_a4_trans">
 			<type>transmission_interface/SimpleTransmission</type>
-			<joint name="${name}_4_joint">
+			<joint name="${name}_a4_joint">
 				<hardwareInterface>${Interface10}</hardwareInterface>
 				<hardwareInterface>${Interface30}</hardwareInterface>
 			</joint>
-			<actuator name="${name}_4_motor">
+			<actuator name="${name}_a4_motor">
 				<mechanicalReduction>1</mechanicalReduction>
 			</actuator>
 		</transmission>
-		<transmission name="${name}_5_trans">
+		<transmission name="${name}_a5_trans">
 			<type>transmission_interface/SimpleTransmission</type>
-			<joint name="${name}_5_joint">
+			<joint name="${name}_a5_joint">
 				<hardwareInterface>${Interface10}</hardwareInterface>
 				<hardwareInterface>${Interface30}</hardwareInterface>
 			</joint>
-			<actuator name="${name}_5_motor">
+			<actuator name="${name}_a5_motor">
 				<mechanicalReduction>1</mechanicalReduction>
 			</actuator>
 		</transmission>
-		<transmission name="${name}_6_trans">
+		<transmission name="${name}_a6_trans">
 			<type>transmission_interface/SimpleTransmission</type>
-			<joint name="${name}_6_joint">
+			<joint name="${name}_a6_joint">
 				<hardwareInterface>${Interface10}</hardwareInterface>
 				<hardwareInterface>${Interface30}</hardwareInterface>
 			</joint>
-			<actuator name="${name}_6_motor">
+			<actuator name="${name}_a6_motor">
 				<mechanicalReduction>1</mechanicalReduction>
 			</actuator>

File: lwr_description/model/kuka_lwr.urdf.xacro (robot description, xacro)
@@ -34,5 +34,5 @@
 				<origin xyz="0 0 0" rpy="0 0 ${M_PI}"/>
 				<geometry>
-					<mesh filename="package://lwr_description/meshes/base.STL"/>
+					<mesh filename="package://lwr_description/meshes/lwr4plus/visual/base.STL"/>
 				</geometry>
 				<material name="Kuka/Orange"/>
@@ -41,5 +41,4 @@
 				<origin xyz="0 0 0.055" rpy="0 0 ${M_PI}"/>
 				<geometry>
-					<!-- <mesh filename="package://lwr_description/meshes/convex/arm_base_convex.stl"/> -->
 					<cylinder radius="0.07" length="0.11"/>
 				</geometry>
@@ -47,5 +46,5 @@
 		</link>
 		<!-- Second segment of the arm. Joint along z-axis -->
-		<joint name="${name}_0_joint" type="revolute">
+		<joint name="${name}_a1_joint" type="revolute">
 			<origin xyz="0 0 0.11" rpy="0 0 0"/>
 			<axis xyz="0 0 1"/>
@@ -55,5 +54,5 @@
 			<child link="${name}_1_link"/>
 		</joint>
-		<joint name="${name}_0_joint_stiffness" type="revolute">
+		<joint name="${name}_a1_joint_stiffness" type="revolute">
 			<axis xyz="0 0 1"/>
 			<limit lower="${min_stiffness}" upper="${max_stiffness}" effort="0" velocity="${rate_stiffness}" />
@@ -72,5 +71,5 @@
 				<origin xyz="0 0 -0.008" rpy="0 0 ${M_PI}"/>
 				<geometry>
-					<mesh filename="package://lwr_description/meshes/link_1.STL"/>
+					<mesh filename="package://lwr_description/meshes/lwr4plus/visual/link_1.STL"/>
 				</geometry>
 				<material name="Kuka/Orange"/>
@@ -79,5 +78,4 @@
 				<origin xyz="0 0 0.0" rpy="0 0 0"/>
 				<geometry>
-					<!--mesh filename="package://lwr_description/meshes/convex/arm_segment_a_convex.stl"/-->
 					<sphere radius="0.07"/>
 				</geometry>
@@ -97,5 +95,5 @@
 		</link>
 		<!-- Third segment of the arm. Joint along y-axis -->
-		<joint name="${name}_1_joint" type="revolute">
+		<joint name="${name}_a2_joint" type="revolute">
 			<origin xyz="0 0 0.2005" rpy="0 0 0"/>
 			<axis xyz="0 -1 0"/>
@@ -105,5 +103,5 @@
 			<child link="${name}_2_link"/>
 		</joint>
-		<joint name="${name}_1_joint_stiffness" type="revolute">
+		<joint name="${name}_a2_joint_stiffness" type="revolute">
 			<axis xyz="0 0 1"/>
 			<limit lower="${min_stiffness}" upper="${max_stiffness}" effort="0" velocity="${rate_stiffness}" />
@@ -122,5 +120,5 @@
 				<origin xyz="0 0 0.0" rpy="0 0 ${M_PI}"/>
 				<geometry>
-					<mesh filename="package://lwr_description/meshes/link_2.STL"/>
+					<mesh filename="package://lwr_description/meshes/lwr4plus/visual/link_2.STL"/>
 				</geometry>
 				<material name="Kuka/Orange"/>
@@ -129,5 +127,4 @@
 				<origin xyz="0 0 0.2" rpy="0 0 0"/>
 				<geometry>
-					<!--mesh filename="package://lwr_description/meshes/convex/arm_segment_b_convex.stl"/-->
 					<sphere radius="0.07"/>
 				</geometry>
@@ -147,5 +144,5 @@
 		</link>
 		<!-- Fourth element of the arm. z-axis -->
-		<joint name="${name}_2_joint" type="revolute">
+		<joint name="${name}_e1_joint" type="revolute">
 			<origin xyz="0 0 0.20" rpy="0 0 0"/>
 			<axis xyz="0 0 1"/>
@@ -155,5 +152,5 @@
 			<child link="${name}_3_link"/>
 		</joint>
-		<joint name="${name}_2_joint_stiffness" type="revolute">
+		<joint name="${name}_e1_joint_stiffness" type="revolute">
 			<axis xyz="0 0 1"/>
 			<limit lower="${min_stiffness}" upper="${max_stiffness}" effort="0" velocity="${rate_stiffness}" />
@@ -172,5 +169,5 @@
 				<origin xyz="0 0 -0.008" rpy="0 0 ${M_PI}"/>
 				<geometry>
-					<mesh filename="package://lwr_description/meshes/link_3.STL"/>
+					<mesh filename="package://lwr_description/meshes/lwr4plus/visual/link_3.STL"/>
 				</geometry>
 				<material name="Kuka/Orange"/>
@@ -179,5 +176,4 @@
 				<origin xyz="0 0 0.0" rpy="0 0 0"/>
 				<geometry>
-					<!--mesh filename="package://lwr_description/meshes/convex/arm_segment_a_convex.stl"/-->
 					<sphere radius="0.07"/>
 				</geometry>
@@ -197,5 +193,5 @@
 		</link>
 		<!-- fifth element of the arm. x-axis -->
-		<joint name="${name}_3_joint" type="revolute">
+		<joint name="${name}_a3_joint" type="revolute">
 			<origin xyz="0 0 0.20" rpy="0 0 0"/>
 			<axis xyz="0 1 0"/>
@@ -205,5 +201,5 @@
 			<child link="${name}_4_link"/>
 		</joint>
-		<joint name="${name}_3_joint_stiffness" type="revolute">
+		<joint name="${name}_a3_joint_stiffness" type="revolute">
 			<axis xyz="0 0 1"/>
 			<limit lower="${min_stiffness}" upper="${max_stiffness}" effort="0" velocity="${rate_stiffness}" />
@@ -222,5 +218,5 @@
 				<origin xyz="0 0 0.0" rpy="0 0 ${M_PI}"/>
 				<geometry>
-					<mesh filename="package://lwr_description/meshes/link_4.STL"/>
+					<mesh filename="package://lwr_description/meshes/lwr4plus/visual/link_4.STL"/>
 				</geometry>
 				<material name="Kuka/Orange"/>
@@ -229,5 +225,4 @@
 			<origin xyz="0 0 0.2" rpy="0 0 0"/>
 			<geometry>
-				<!--mesh filename="package://lwr_description/meshes/convex/arm_segment_b_convex.stl"/-->
 				<sphere radius="0.07"/>
 			</geometry>
@@ -247,5 +242,5 @@
 		</link>
 		<!-- Sixth element of the arm. z-axis -->
-		<joint name="${name}_4_joint" type="revolute">
+		<joint name="${name}_a4_joint" type="revolute">
 			<origin xyz="0 0 0.20" rpy="0 0 0"/>
 			<axis xyz="0 0 1"/>
@@ -255,5 +250,5 @@
 			<child link="${name}_5_link"/>
 		</joint>
-		<joint name="${name}_4_joint_stiffness" type="revolute">
+		<joint name="${name}_a4_joint_stiffness" type="revolute">
 			<axis xyz="0 0 1"/>
 			<limit lower="${min_stiffness}" upper="${max_stiffness}" effort="0" velocity="${rate_stiffness}" />
@@ -272,5 +267,5 @@
 				<origin xyz="0 0 -0.008" rpy="0 0 ${M_PI}"/>
 				<geometry name="${name}_5_geom">
-					<mesh filename="package://lwr_description/meshes/link_5.STL"/>
+					<mesh filename="package://lwr_description/meshes/lwr4plus/visual/link_5.STL"/>
 				</geometry>
 				<material name="Kuka/Orange"/>
@@ -279,5 +274,4 @@
 				<origin xyz="0 0 0.0" rpy="0 0 0"/>
 				<geometry>
-					<!--mesh filename="package://lwr_description/meshes/convex/arm_segment_last_convex.stl"/-->
 					<sphere radius="0.07"/>
 				</geometry>
@@ -297,5 +291,5 @@
 		</link>
 		<!-- Seventh element of the arm. z-axis -->
-		<joint name="${name}_5_joint" type="revolute">
+		<joint name="${name}_a5_joint" type="revolute">
 			<origin xyz="0 0 0.19" rpy="0 0 0"/>
 			<axis xyz="0 -1 0"/>
@@ -305,5 +299,5 @@
 			<child link="${name}_6_link"/>
 		</joint>
-		<joint name="${name}_5_joint_stiffness" type="revolute">
+		<joint name="${name}_a5_joint_stiffness" type="revolute">
 			<axis xyz="0 0 1"/>
 			<limit lower="${min_stiffness}" upper="${max_stiffness}" effort="0" velocity="${rate_stiffness}" />
@@ -322,17 +316,17 @@
 				<origin xyz="0 0 0" rpy="0 0 ${M_PI}"/>
 				<geometry>
-					<mesh filename="package://lwr_description/meshes/link_6.STL"/>
+					<mesh filename="package://lwr_description/meshes/lwr4plus/visual/link_6.STL"/>
 				</geometry>
 			<material name="Kuka/Grey"/>
 			</visual>
 			<collision>
-			<origin xyz="0 0 0" rpy="0 0 ${M_PI}"/>
+			<origin xyz="0 -0.01 0" rpy="0 0 ${M_PI}"/>
 			<geometry>
-				<mesh filename="package://lwr_description/meshes/convex/arm_wrist_convex.stl"/>
+				<sphere radius="0.08"/>
 			</geometry>
 			</collision>
 		</link>
 		<!-- Eighth element of the arm. z-axis -->
-		<joint name="${name}_6_joint" type="revolute">
+		<joint name="${name}_a6_joint" type="revolute">
 			<origin xyz="0 0 0.078" rpy="0 0 0"/>
 			<axis xyz="0 0 1"/>
@@ -342,5 +336,5 @@
 			<child link="${name}_7_link"/>
 		</joint>
-		<joint name="${name}_6_joint_stiffness" type="revolute">
+		<joint name="${name}_a6_joint_stiffness" type="revolute">
 			<axis xyz="0 0 1"/>
 			<limit lower="${min_stiffness}" upper="${max_stiffness}" effort="0" velocity="${rate_stiffness}" />
@@ -359,5 +353,5 @@
 				<origin xyz="0 0 0" rpy="0 0 ${M_PI}"/>
 				<geometry>
-					<mesh filename="package://lwr_description/meshes/link_7.STL"/>
+					<mesh filename="package://lwr_description/meshes/lwr4plus/visual/link_7.STL"/>
 				</geometry>
 			<material name="Kuka/DarkGrey"/>
