Commit message: Just a change for trying to add the contact sensor on fingertips

File: single_lwr_example/single_lwr_robot/robot/lwr_adaptive.urdf.xacro (robot description, xacro)
@@ -3,6 +3,6 @@
   <!-- MODELS -->
   <xacro:include filename="$(find lwr_description)/model/kuka_lwr.urdf.xacro"/>
-  <xacro:include filename="$(find soft_hand_description)/model/soft_hand.urdf.xacro"/>
-  <!-- <xacro:include filename="$(find soft_hand_description)/model/soft_hand_soma_ocado.urdf.xacro"/> -->
+  <!-- <xacro:include filename="$(find soft_hand_description)/model/soft_hand_contact_distal.urdf.xacro"/> -->
+  <xacro:include filename="$(find soft_hand_description)/model/soft_hand_soma_ocado.urdf.xacro"/>
   <link name="world"/>
   <!-- RIGHT ARM -->
@@ -24,7 +24,7 @@
   </gazebo>
   <!-- RIGHT SOFTHAND -->
-  <xacro:soft_hand parent="right_arm_7_link" name="right_hand" left="false" withAdaptiveTransmission="true" useMimicTag="$(arg use_mimic_tag)">
+  <xacro:soft_hand_soma_ocado parent="right_arm_7_link" name="right_hand" left="false" withAdaptiveTransmission="true" useMimicTag="$(arg use_mimic_tag)">
     <origin xyz="0 0 0" rpy="0 0 3.1415"/>
-  </xacro:soft_hand>
+  </xacro:soft_hand_soma_ocado>
   <!-- EXTRA ENDEFFECTOR -->
   <joint name="right_hand_ee_joint" type="fixed">
@@ -40,7 +40,7 @@
   <sensor name="thumb_distal_link_contact_sensor" type="contact">
     <always_on>true</always_on>
-    <update_rate>30.0</update_rate>
+    <update_rate>10.0</update_rate>
     <contact>
-      <collision>collision</collision>
+      <collision>right_hand_thumb_distal_link_collision_collision</collision>
     </contact>
     <plugin name="gripper_bumper" filename="libgazebo_ros_bumper.so">
