Commit message: importing single_lwr_example packages, moving lwr_launch -> single_lwr_launch, deleting lwr_moveit it will become single_lwr_moveit, cleaning some license headers, package.xml, CMakeLists.txt, etc

File: single_lwr_example/single_lwr_robot/robot/single_lwr_robot.urdf.xacro (robot description, xacro)
@@ -1,6 +1,16 @@
 <?xml version="1.0"?>
-<robot xmlns:xacro="http://www.ros.org/wiki/xacro" name="lwr">
+<robot xmlns:xacro="http://www.ros.org/wiki/xacro" name="single_lwr_robot">
+	<!-- Include all models -->
 	<xacro:include filename="$(find lwr_description)/model/kuka_lwr.urdf.xacro"/>
+	<!-- and assemble your robot -->
 	<link name="world">
+		<inertial>
+			<mass value="5.0"/>
+			<origin rpy="0 0 0" xyz="0 0 0"/>
+			<inertia ixx="0.01"
+             iyy="0.01"
+             izz="0.01"
+             ixy="0" iyz="0" ixz="0"/>
+		</inertial>
 		<visual>
 			<origin xyz="0 0 0.50" rpy="0 0 0"/>
@@ -19,4 +29,5 @@
 		<static>true</static>>
 	</gazebo>
+	<!-- using the models -->
 	<xacro:kuka_lwr parent="world" name="lwr">
 		<origin xyz="0 0 1" rpy="0 0 0"/>

Commit message: Importing single_lwr_moveit, and update on several README files.

File: single_lwr_example/single_lwr_robot/robot/single_lwr_robot.urdf.xacro (robot description, xacro)
@@ -4,5 +4,5 @@
 	<xacro:include filename="$(find lwr_description)/model/kuka_lwr.urdf.xacro"/>
 	<!-- and assemble your robot -->
-	<link name="world">
+	<link name="box">
 		<inertial>
 			<mass value="5.0"/>
@@ -26,9 +26,9 @@
 		</collision>
 	</link>
-	<gazebo reference="world">
+	<gazebo reference="box">
 		<static>true</static>>
 	</gazebo>
 	<!-- using the models -->
-	<xacro:kuka_lwr parent="world" name="lwr">
+	<xacro:kuka_lwr parent="box" name="lwr">
 		<origin xyz="0 0 1" rpy="0 0 0"/>
 	</xacro:kuka_lwr>

Commit message: Add fixed joint world->box so that the robot doesn't wiggle

File: single_lwr_example/single_lwr_robot/robot/single_lwr_robot.urdf.xacro (robot description, xacro)
@@ -4,4 +4,10 @@
 	<xacro:include filename="$(find lwr_description)/model/kuka_lwr.urdf.xacro"/>
 	<!-- and assemble your robot -->
+    <link name="world" />
+    <joint name="fixed" type="fixed">
+        <origin xyz="0 0 0" rpy="0 0 0"/>
+        <parent link="world"/>
+        <child link="box"/>
+    </joint>
 	<link name="box">
 		<inertial>

Commit message: Remove world link, keep box out of kinematic chain (against wiggling)

File: single_lwr_example/single_lwr_robot/robot/single_lwr_robot.urdf.xacro (robot description, xacro)
@@ -4,10 +4,4 @@
 	<xacro:include filename="$(find lwr_description)/model/kuka_lwr.urdf.xacro"/>
 	<!-- and assemble your robot -->
-    <link name="world" />
-    <joint name="fixed" type="fixed">
-        <origin xyz="0 0 0" rpy="0 0 0"/>
-        <parent link="world"/>
-        <child link="box"/>
-    </joint>
 	<link name="box">
 		<inertial>

Commit message: Removed box

File: single_lwr_example/single_lwr_robot/robot/single_lwr_robot.urdf.xacro (robot description, xacro)
@@ -3,33 +3,8 @@
 	<!-- Include all models -->
 	<xacro:include filename="$(find lwr_description)/model/kuka_lwr.urdf.xacro"/>
-	<!-- and assemble your robot -->
-	<link name="box">
-		<inertial>
-			<mass value="5.0"/>
-			<origin rpy="0 0 0" xyz="0 0 0"/>
-			<inertia ixx="0.01"
-             iyy="0.01"
-             izz="0.01"
-             ixy="0" iyz="0" ixz="0"/>
-		</inertial>
-		<visual>
-			<origin xyz="0 0 0.50" rpy="0 0 0"/>
-			<geometry>
-				<box size="1.0 1.0 1.0"/>
-			</geometry>
-		</visual>
-		<collision>
-			<origin xyz="0 0 0.50" rpy="0 0 0"/>
-			<geometry>
-				<box size="1.0 1.0 1.0"/>
-			</geometry>
-		</collision>
-	</link>
-	<gazebo reference="box">
-		<static>true</static>>
-	</gazebo>
+	<link name="world"/>
 	<!-- using the models -->
-	<xacro:kuka_lwr parent="box" name="lwr">
-		<origin xyz="0 0 1" rpy="0 0 0"/>
+	<xacro:kuka_lwr parent="world" name="lwr">
+		<origin xyz="0 0 0" rpy="0 0 0"/>
 	</xacro:kuka_lwr>
 </robot>
